File: Circuit/ControlCircuit.kicad_pcb (KiCad board)
At the start: 2 copper layers, 4 parts, among them IC1 ATMEGA328-P, K1 Meisei-m4-24h

Commit message: Continued PCB work, placement started. Report and presentation also started
Parts:
- removed IC1: ATMEGA328-P, Housings_DIP:DIP-28_W7.62mm
- removed K1: Meisei-m4-24h, Meisei:Meisei-m4-24h
- removed LCD1: tft-proto-mi0283qt-9a, Pin_Headers:Pin_Header_Straight_2x20_Pitch2.54mm
- removed R1: 100R, Resistors_SMD:R_0805
- added C101: 4uF, Capacitors_SMD:C_0805, F.Cu at (121.9, 39.4)
- added C102: 32pF, Capacitors_SMD:C_0805, F.Cu at (121.9, 34.3)
- added C103: 100uF, Capacitors_SMD:C_0805, F.Cu at (137.2, 31.8)
- added D101: D_Schottky, Diodes_SMD:D_0805, F.Cu at (121.9, 31.8)
- added D201: D, Diodes_SMD:D_0805, F.Cu at (22.9, 53.3)
- added D202: D, Diodes_SMD:D_0805, F.Cu at (39.4, 53.3)
- added D203: D, Diodes_SMD:D_0805, F.Cu at (55.9, 53.3)
- added D204: D, Diodes_SMD:D_0805, F.Cu at (72.4, 53.3)
- added D205: D, Diodes_SMD:D_0805, F.Cu at (88.9, 53.3)
- added D206: D, Diodes_SMD:D_0805, F.Cu at (105.4, 53.3)
- added IC101: ATMEGA328-P, Housings_DIP:DIP-28_W7.62mm, F.Cu at (120.7, 87.6)
- added K201: Meisei-m4-24h, Meisei:Meisei-m4-24h, F.Cu at (19.1, 57.1)
- added K202: Meisei-m4-24h, Meisei:Meisei-m4-24h, F.Cu at (35.6, 57.1)
- added K203: Meisei-m4-24h, Meisei:Meisei-m4-24h, F.Cu at (52.1, 56.9)
- added K204: Meisei-m4-24h, Meisei:Meisei-m4-24h, F.Cu at (68.5, 56.9)
- added K205: Meisei-m4-24h, Meisei:Meisei-m4-24h, F.Cu at (84.9, 56.9)
- added K206: Meisei-m4-24h, Meisei:Meisei-m4-24h, F.Cu at (101.3, 56.9)
- added K301: Meisei-m4-24h, Meisei:Meisei-m4-24h, F.Cu at (92.1, 142.9)
- added K302: Meisei-m4-24h, Meisei:Meisei-m4-24h, F.Cu at (79.5, 142.9)
- added K303: Meisei-m4-24h, Meisei:Meisei-m4-24h, F.Cu at (66.9, 142.9)
- added K304: Meisei-m4-24h, Meisei:Meisei-m4-24h, F.Cu at (54.3, 142.9)
- added K305: Meisei-m4-24h, Meisei:Meisei-m4-24h, F.Cu at (41.7, 142.9)
- added K306: Meisei-m4-24h, Meisei:Meisei-m4-24h, F.Cu at (29.2, 142.9)
- added L101: 260mH, Inductors:Inductor_1212, F.Cu at (127.0, 41.9)
- added LCD101: tft-proto-mi0283qt-9a, Pin_Headers:Pin_Header_Straight_2x20_Pitch2.54mm, F.Cu at (21.6, 83.8)
- added Q201: Q_NPN_BCE, MMBT3904:MMBT3904, F.Cu at (15.2, 59.7)
- added Q202: Q_NPN_BCE, MMBT3904:MMBT3904, F.Cu at (31.8, 59.7)
- added Q203: Q_NPN_BCE, MMBT3904:MMBT3904, F.Cu at (48.3, 59.7)
- added Q204: Q_NPN_BCE, MMBT3904:MMBT3904, F.Cu at (64.8, 59.7)
- added Q205: Q_NPN_BCE, MMBT3904:MMBT3904, F.Cu at (81.3, 59.7)
- added Q206: Q_NPN_BCE, MMBT3904:MMBT3904, F.Cu at (97.8, 59.7)
- added R101: 18kR, Resistors_SMD:R_0805, F.Cu at (133.3, 40.6)
- added R102: 11kR, Resistors_SMD:R_0805, F.Cu at (137.2, 36.8)
- added R103: 1.5R, Resistors_SMD:R_0805, F.Cu at (137.2, 27.9)
- added R104: 100R, Resistors_SMD:R_0805, F.Cu at (27.9, 85.1)
- added R201: 10kR, Resistors_SMD:R_0805, F.Cu at (14.0, 64.8)
- added R202: 10kR, Resistors_SMD:R_0805, F.Cu at (30.5, 64.8)
- added R203: 10kR, Resistors_SMD:R_0805, F.Cu at (47.0, 64.8)
- added R204: 10kR, Resistors_SMD:R_0805, F.Cu at (63.5, 64.8)
- added R205: 10kR, Resistors_SMD:R_0805, F.Cu at (80.0, 64.8)
- added R206: 10kR, Resistors_SMD:R_0805, F.Cu at (96.5, 64.8)
- added VR101: MC34063A, Housings_DIP:DIP-8_W7.62mm, F.Cu at (125.7, 29.2)
Other:
- board text added: "Screen circuit board outline"

Commit message: Continued PCB work, additional footprints added
Parts:
- removed IC101: ATMEGA328-P, Housings_DIP:DIP-28_W7.62mm
- removed LCD101: tft-proto-mi0283qt-9a, Pin_Headers:Pin_Header_Straight_2x20_Pitch2.54mm
- removed R104: 100R, Resistors_SMD:R_0805
- added C501: C, Capacitors_SMD:C_0805, F.Cu at (78.7, 100.3)
- added C502: C, Capacitors_SMD:C_0805, F.Cu at (78.7, 95.2)
- added CON501: AVR-ISP-10, Connectors:IDC_Header_Straight_10pins, F.Cu at (114.3, 111.8)
- added IC501: ATMEGA644-A, Housings_QFP:LQFP-44_10x10mm_Pitch0.8mm, F.Cu at (57.1, 97.8)
- added LCD401: tft-proto-mi0283qt-9a, Pin_Headers:Pin_Header_Straight_2x20_Pitch2.54mm, F.Cu at (20.3, 82.5)
- added R401: 100R, Resistors_SMD:R_0805, F.Cu at (26.7, 83.8)
- added Y501: Crystal, Crystals:Crystal_HC49-U_Vertical, F.Cu at (72.4, 100.3)
Connections:
- net Output1 renamed /RelayOutputs/O1
- net Output2 renamed /RelayOutputs/O2
- net Output3 renamed /RelayOutputs/O3
- net Output4 renamed /RelayOutputs/O4
- net Output5 renamed /RelayOutputs/O5
- net Output6 renamed /RelayOutputs/O6
- net RelayOutput1 renamed /RelayOutputs/OR1sel2
- net RelayOutput2 renamed /RelayOutputs/OR2sel2
- net RelayOutput3 renamed /RelayOutputs/OR3sel2
- net RelayOutput4 renamed /RelayOutputs/OR4sel2
- net RelayOutput5 renamed /RelayOutputs/OR5sel2
- net RelayOutput6 renamed /RelayOutputs/OR6sel2
- K201 pad 4: GNDREF -> /RelayOutputs/OR1com
- K201 pad 6: GNDREF -> /RelayOutputs/OR1sel1
- K202 pad 4: GNDREF -> /RelayOutputs/OR2com
- K202 pad 6: GNDREF -> /RelayOutputs/OR2sel1
- K203 pad 4: GNDREF -> /RelayOutputs/OR3com
- K203 pad 6: GNDREF -> /RelayOutputs/OR3sel1
- K204 pad 4: GNDREF -> /RelayOutputs/OR4com
- K204 pad 6: GNDREF -> /RelayOutputs/OR4sel1
- K205 pad 4: GNDREF -> /RelayOutputs/OR5com
- K205 pad 6: GNDREF -> /RelayOutputs/OR5sel1
- K206 pad 4: GNDREF -> /RelayOutputs/OR6com
- K206 pad 6: GNDREF -> /RelayOutputs/OR6sel1

Commit message: Additional PCB work
Parts:
- added D207: D, Diodes_SMD:D_MiniMELF_Standard, F.Cu at (144.8, 72.4)
- added D208: D, Diodes_SMD:D_MiniMELF_Standard, F.Cu at (156.2, 72.4)
- added K207: Meisei-m4-24h, Meisei:Meisei-m4-24h, F.Cu at (148.6, 69.2)
- added K208: Meisei-m4-24h, Meisei:Meisei-m4-24h, F.Cu at (160.0, 69.2)
- added K307: Meisei-m4-24h, Meisei:Meisei-m4-24h, F.Cu at (141.0, 138.4)
- added K308: Meisei-m4-24h, Meisei:Meisei-m4-24h, F.Cu at (152.4, 138.4)
- added P101: CONN_01X08, Connectors_Terminal_Blocks:TerminalBlock_Pheonix_MKDS1.5-8pol, F.Cu at (167.6, 123.2)
- added P102: CONN_01X08, Connectors_Terminal_Blocks:TerminalBlock_Pheonix_MKDS1.5-8pol, F.Cu at (168.3, 77.5)
- added P103: CONN_01X08, Connectors_Terminal_Blocks:TerminalBlock_Pheonix_MKDS1.5-8pol, F.Cu at (148.0, 44.5)
- added P104: CONN_01X08, Connectors_Terminal_Blocks:TerminalBlock_Pheonix_MKDS1.5-8pol, F.Cu at (106.7, 44.5)
- added P105: CONN_01X02, Connectors_Terminal_Blocks:TerminalBlock_Pheonix_MKDS1.5-2pol, F.Cu at (167.6, 109.9)
- added Q207: Q_NPN_BCE, MMBT3904:MMBT3904, F.Cu at (147.3, 76.8)
- added Q208: Q_NPN_BCE, MMBT3904:MMBT3904, F.Cu at (158.1, 76.8)
- added R207: 10kR, Resistors_SMD:R_0805, F.Cu at (142.2, 77.5)
- added R208: 10kR, Resistors_SMD:R_0805, F.Cu at (153.0, 77.5)
- D101, D201, D202, D203, D204, D205, D206: footprint Diodes_SMD:D_0805 -> Diodes_SMD:D_MiniMELF_Standard
- L101: footprint Inductors:Inductor_1212 -> Inductors:Inductor_Wurth_HCI-7050
- VR101: footprint Housings_DIP:DIP-8_W7.62mm -> Housings_SOIC:SOIC-8_3.9x4.9mm_Pitch1.27mm
- moved K306 100.5 mm to (129.5, 138.4)
- moved K305 76.5 mm to (118.1, 138.4)
- moved VR101 67.5 mm to (136.5, 95.9)
- moved C103 66.3 mm to (143.5, 97.8), turned to 270 degrees
- moved Q201 65.8 mm to (78.7, 76.8)
- moved R102 65.1 mm to (143.5, 101.6), turned to 270 degrees
- moved R103 65.1 mm to (143.5, 92.7)
- moved R101 64.7 mm to (142.2, 104.8)
- moved L101 63.5 mm to (135.9, 104.8)
- moved C101 63.3 mm to (129.5, 102.2)
- moved C102 63.2 mm to (128.3, 97.2)
- moved K201 62.8 mm to (80.6, 69.2), turned to 180 degrees
- moved D101 61.9 mm to (127.6, 93.3)
- moved R201 61.0 mm to (73.7, 77.5), turned to 180 degrees
- moved Q202 60.9 mm to (90.2, 76.8)
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Connections:
- CON501 pad 5: /Microcontroller/RST -> /LCDTouchScreen/RST
- IC501 pad 10: Net-(IC501-Pad10) -> /RelayInputs/I2
- IC501 pad 11: Net-(IC501-Pad11) -> /RelayInputs/I3
- IC501 pad 12: Net-(IC501-Pad12) -> /RelayInputs/I4
- IC501 pad 13: Net-(IC501-Pad13) -> /RelayInputs/I5
- IC501 pad 14: Net-(IC501-Pad14) -> /RelayInputs/I6
- IC501 pad 15: Net-(IC501-Pad15) -> /RelayInputs/I7
- IC501 pad 16: Net-(IC501-Pad16) -> /RelayInputs/I8
- IC501 pad 19: Net-(IC501-Pad19) -> /RelayOutputs/O8
- IC501 pad 20: Net-(IC501-Pad20) -> /RelayOutputs/O7
- IC501 pad 21: Net-(IC501-Pad21) -> /RelayOutputs/O6
- IC501 pad 22: Net-(IC501-Pad22) -> /RelayOutputs/O5
- IC501 pad 23: Net-(IC501-Pad23) -> /RelayOutputs/O4
- IC501 pad 24: Net-(IC501-Pad24) -> /RelayOutputs/O3
- IC501 pad 25: Net-(IC501-Pad25) -> /RelayOutputs/O2
- IC501 pad 26: Net-(IC501-Pad26) -> /RelayOutputs/O1
- IC501 pad 34: /Microcontroller/ADC3 -> /Microcontroller/ADC0
- IC501 pad 35: /Microcontroller/ADC2 -> /Microcontroller/ADC1
- IC501 pad 36: /Microcontroller/ADC1 -> /Microcontroller/ADC2
- IC501 pad 37: /Microcontroller/ADC0 -> /Microcontroller/ADC3
- IC501 pad 4: /Microcontroller/RST -> /LCDTouchScreen/RST
- IC501 pad 42: Net-(IC501-Pad42) -> /LCDTouchScreen/WR
- IC501 pad 43: Net-(IC501-Pad43) -> /LCDTouchScreen/CS
- IC501 pad 44: Net-(IC501-Pad44) -> /LCDTouchScreen/RST
- IC501 pad 9: Net-(IC501-Pad9) -> /RelayInputs/I1
- K206 pad 6: /RelayOutputs/OR6sel1 -> /OR6s1
- K206 pad 8: /RelayOutputs/OR6sel2 -> /OR6s2
- K301 pad 16: RelayInput1 -> /RelayInputs/RI1
- K301 pad 4: Input1 -> /RelayInputs/I1
- K302 pad 16: RelayInput2 -> /RelayInputs/RI2
- K302 pad 4: Input2 -> /RelayInputs/I2
- K303 pad 16: RelayInput3 -> /RelayInputs/RI3
- K303 pad 4: Input3 -> /RelayInputs/I3
- K304 pad 16: RelayInput4 -> /RelayInputs/RI4
- K304 pad 4: Input4 -> /RelayInputs/I4
- K305 pad 16: RelayInput5 -> /RelayInputs/RI5
- K305 pad 4: Input5 -> /RelayInputs/I5
- K306 pad 16: RelayInput6 -> /RelayInputs/RI6
- K306 pad 4: Input6 -> /RelayInputs/I6
Other:
- board outline added: 106.7 x 121.9 mm
