File: Circuit/ControlCircuit.kicad_pcb (KiCad board)
At the start: 2 copper layers, 120 x 120 mm, 123 parts, among them CON501 AVR-ISP-10, IC501 ATMEGA644-A, K201 Meisei-m4-24h, K202 Meisei-m4-24h, K203 Meisei-m4-24h, K204 Meisei-m4-24h, K205 Meisei-m4-24h, K206 Meisei-m4-24h, K207 Meisei-m4-24h, K208 Meisei-m4-24h, P101 CONN_01X08, P102 CONN_01X08, P103 CONN_01X08, P104 CONN_01X08, P105 CONN_01X08, P106 CONN_01X08, P107 CONN_01X02, Q201 Q_NPN_BCE, Q202 Q_NPN_BCE, Q203 Q_NPN_BCE, Q204 Q_NPN_BCE, Q205 Q_NPN_BCE, Q206 Q_NPN_BCE, Q207 Q_NPN_BCE, Q208 Q_NPN_BCE, U301 LTV-817, U302 LTV-817, U303 LTV-817, U304 LTV-817, U305 LTV-817, U306 LTV-817, U307 LTV-817, U308 LTV-817, Y501 Crystal

Commit message: Report writing
Connections:
- D101 pad 1: +3V3 -> Net-(D101-Pad1)
- L101 pad 2: Net-(L101-Pad2) -> Net-(D101-Pad1)
- R101 pad 2: Net-(L101-Pad2) -> +3V3
- VR101 pad 2: +3V3 -> Net-(D101-Pad1)
Routing:
- net Net-(D101-Pad1): track 0.00 -> 6.62 mm, vias 0 -> 2
- net +3V3: track 189.4 -> 185.6 mm, vias 17 -> 15
- net Net-(L101-Pad2): track 2.85 -> 0.00 mm
